File: ELE305_display.kicad_sch (KiCad schematic)
At the start: 20 parts, among them J2 687124182122

Commit message: Updated PCB
Parts:
- removed TP1: VDD_3.0V, TestPoint:TestPoint_Pad_D1.5mm, symbol Connector:TestPoint
- removed TP11: P11, TestPoint:TestPoint_Pad_D1.5mm, symbol Connector:TestPoint
- removed TP12: P12, TestPoint:TestPoint_Pad_D1.5mm, symbol Connector:TestPoint
- removed TP17: P17, TestPoint:TestPoint_Pad_D1.5mm, symbol Connector:TestPoint
- removed TP18: P18, TestPoint:TestPoint_Pad_D1.5mm, symbol Connector:TestPoint
- removed TP19: P19, TestPoint:TestPoint_Pad_D1.5mm, symbol Connector:TestPoint
- removed TP20_10_7_1: ground, TestPoint:TestPoint_Pad_D1.5mm, symbol Connector:TestPoint
- removed TP21: P21, TestPoint:TestPoint_Pad_D1.5mm, symbol Connector:TestPoint
- removed TP22: P22, TestPoint:TestPoint_Pad_D1.5mm, symbol Connector:TestPoint
- removed TP23: P23, TestPoint:TestPoint_Pad_D1.5mm, symbol Connector:TestPoint
- removed TP24: P24, TestPoint:TestPoint_Pad_D1.5mm, symbol Connector:TestPoint
- removed TP4: P4, TestPoint:TestPoint_Pad_D1.5mm, symbol Connector:TestPoint
- removed TP5: P5, TestPoint:TestPoint_Pad_D1.5mm, symbol Connector:TestPoint
- removed TP6: SDIO, TestPoint:TestPoint_Pad_D1.5mm, symbol Connector:TestPoint
- removed TP8: P8, TestPoint:TestPoint_Pad_D1.5mm, symbol Connector:TestPoint
- removed TP9: P9, TestPoint:TestPoint_Pad_D1.5mm, symbol Connector:TestPoint
- added J1: Conn_01x16_Pin, Connector_PinHeader_2.54mm:PinHeader_1x16_P2.54mm_Vertical, symbol Connector:Conn_01x16_Pin
Connections:
- net GND: now also J1.12 (Pin_12)
- net at R6.1: now also J1.4 (Pin_4)
- net at J2.12: now also J1.8 (Pin_8)
- net at J2.19: now also J1.11 (Pin_11)
- net at C1.2, C2.2, J2.2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: now also J1.1 (Pin_1)
- net at J2.4: now also J1.2 (Pin_2)
- net at J2.9: now also J1.6 (Pin_6)
- net at J2.5: now also J1.3 (Pin_3)
- net at J2.17: now also J1.9 (Pin_9)
- net at J2.23: now also J1.15 (Pin_15)
- net at J2.21: now also J1.13 (Pin_13)
- net at J2.11: now also J1.7 (Pin_7)
- net at J2.18: now also J1.10 (Pin_10)
- net at J2.22: now also J1.14 (Pin_14)
- net at J2.24: now also J1.16 (Pin_16)
- net at J2.8: now also J1.5 (Pin_5)

Commit message: last commit
Connections:
- net GND: now also J2.MP1, J2.MP2
- no-connect marks 6 -> 4
Changed lines of the file:
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@@
+	)
+	(junction
+		(at 260.35 254)
+		(diameter 0)
+		(color 0 0 0 0)
+	)
+	(junction
+		(at 355.6 330.2)
+		(diameter 0)
+		(color 0 0 0 0)
 	)
 	(junction
@@
 	)
 	(no_connect
-		(at 355.6 330.2)
-	)
-	(no_connect
 		(at 327.66 304.8)
-	)
-	(no_connect
-		(at 358.14 330.2)
 	)
 	(no_connect
@@
 	(wire
 		(pts
+			(xy 260.35 330.2) (xy 260.35 254)
+		)
+		(stroke
+			(width 0)
+			(type default)
+		)
+	)
+	(wire
+		(pts
 			(xy 508 303.53) (xy 546.1 303.53)
 		)
@@
 	(wire
 		(pts
+			(xy 355.6 330.2) (xy 260.35 330.2)
+		)
+		(stroke
+			(width 0)
+			(type default)
+		)
+	)
+	(wire
+		(pts
 			(xy 101.6 279.4) (xy 101.6 43.18)
 		)
@@
 	(wire
 		(pts
-			(xy 177.8 254) (xy 309.88 254)
+			(xy 177.8 254) (xy 260.35 254)
+		)
+		(stroke
+			(width 0)
+			(type default)
+		)
+	)
+	(wire
+		(pts
+			(xy 260.35 254) (xy 309.88 254)
 		)
 		(stroke
@@
 		)
 		(stroke
+			(width 0)
+			(type default)
+		)
+	)
+	(wire
+		(pts
+			(xy 358.14 330.2) (xy 355.6 330.2)
+		)
+		(stroke
